File: HW/i2cExplorer/i2cExplorer.kicad_pcb (KiCad board)
At the start: 2 copper layers, 38 x 38 mm, 19 parts, among them J1 GC9A01, J2 SWDIO, J3 I2CTest, J4 USB_C_Receptacle, Q1 S8050, SW1 SW_Push, SW2 SW_Push, SW3 SW_Push, U1 RP2040, U2 W5Q16JVSSIQ, Y1 Crystal

Commit message: update sch
Parts:
- moved SW3 3.40 mm to (0.00, 19.0)
- moved H4 2.75 mm to (16.6, -9.65)
- moved U2 2.15 mm to (0.10, 10.7)
- moved H1 2.06 mm to (-16.3, -8.84)
- moved H2 2.02 mm to (-16.3, 8.84)
- moved SW2 1.99 mm to (10.7, -15.6)
- moved SW1 1.97 mm to (-10.7, -15.6)
- moved J3 1.83 mm to (16.2, -3.81)
- moved H3 1.73 mm to (16.2, 8.08)
Other:
- board size 38 x 38 mm -> 42 x 42 mm
Changed lines of the file:
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@@
   )
   (footprint "MountingHole:MountingHole_2.2mm_M2" (layer "F.Cu")
-    (at 14.3256 -8.128)
+    (at 16.6116 -9.652)
     (descr "Mounting Hole 2.2mm, no annular, M2")
     (tags "mounting hole 2.2mm no annular m2")
@@
         (effects (font (size 1 1) (thickness 0.15)))
     )
-    (fp_text user "${REFERENCE}" (at 0 0) (layer "F.Fab")
+    (fp_text user "${REFERENCE}" (at -0.3556 -0.1524) (layer "F.Fab")
         (effects (font (size 1 1) (thickness 0.15)))
     )
@@
   )
   (footprint "Button_Switch_SMD:Panasonic_EVQPUM_EVQPUD" (layer "F.Cu")
-    (at -9.466812 -14.068424 35)
+    (at -10.722623 -15.586866 35)
     (descr "http://industrial.panasonic.com/cdbs/www-data/pdf/ATV0000/ATV0000CE5.pdf")
     (tags "SMD SMT SPST EVQPUM EVQPUD")
@@
   )
   (footprint "MountingHole:MountingHole_2.2mm_M2" (layer "F.Cu")
-    (at -14.4272 7.9756)
+    (at -16.256 8.8392)
     (descr "Mounting Hole 2.2mm, no annular, M2")
     (tags "mounting hole 2.2mm no annular m2")
@@
   )
   (footprint "MountingHole:MountingHole_2.2mm_M2" (layer "F.Cu")
-    (at -14.6812 -7.5692)
+    (at -16.3068 -8.8392)
     (descr "Mounting Hole 2.2mm, no annular, M2")
     (tags "mounting hole 2.2mm no annular m2")
@@
   )
   (footprint "Package_SO:SOIC-8_5.23x5.23mm_P1.27mm" (layer "F.Cu")
-    (at 0.3556 8.5852 180)
+    (at 0.1016 10.7188 180)
     (descr "SOIC, 8 Pin (http://www.winbond.com/resource-files/w25q32jv%20revg%2003272018%20plus.pdf#page=68), generated with kicad-footprint-generator ipc_gullwing_generator.py")
     (tags "SOIC SO")
@@
     (pad "8" smd roundrect (at 3.6 -1.905 180) (size 1.6 0.6) (layers "F.Cu" "F.Paste" "F.Mask") (roundrect_rratio 0.25)
       (net 99 "unconnected-(U2-VCC-Pad8)") (pinfunction "VCC") (pintype "power_in"))
-    (model "${KICAD6_3DMODEL_DIR}/Package_SO.3dshapes/SOIC-8_5.23x5.23mm_P1.27mm.wrl"
+    (model "${KICAD7_3DMODEL_DIR}/Package_SO.3dshapes/SOIC-8_5.275x5.275mm_P1.27mm.step"
       (offset (xyz 0 0 0))
       (scale (xyz 1 1 1))
@@
   )
   (footprint "Button_Switch_SMD:Panasonic_EVQPUM_EVQPUD" (layer "F.Cu")
-    (at 0 15.5922 180)
+    (at 0 18.9958 180)
     (descr "http://industrial.panasonic.com/cdbs/www-data/pdf/ATV0000/ATV0000CE5.pdf")
     (tags "SMD SMT SPST EVQPUM EVQPUD")
@@
   )
   (footprint "MountingHole:MountingHole_2.2mm_M2" (layer "F.Cu")
-    (at 14.4272 8.0264)
+    (at 16.1544 8.0772)
     (descr "Mounting Hole 2.2mm, no annular, M2")
     (tags "mounting hole 2.2mm no annular m2")
@@
     (pad "3" smd rect (at 0.875 -0.7 180) (size 1.15 1) (layers "F.Cu" "F.Paste" "F.Mask"))
     (pad "4" smd rect (at -0.875 -0.7 180) (size 1.15 1) (layers "F.Cu" "F.Paste" "F.Mask"))
-    (model "${KICAD6_3DMODEL_DIR}/Crystal.3dshapes/Crystal_SMD_2520-4Pin_2.5x2.0mm.wrl"
+    (model "${KICAD7_3DMODEL_DIR}/Crystal.3dshapes/Crystal_SMD_Abracon_ABM8G-4Pin_3.2x2.5mm.step"
       (offset (xyz 0 0 0))
       (scale (xyz 1 1 1))
@@
   )
   (footprint "Button_Switch_SMD:Panasonic_EVQPUM_EVQPUD" (layer "F.Cu")
-    (at 9.3472 -14.1732 -35)
+    (at 10.742932 -15.586866 -35)
     (descr "http://industrial.panasonic.com/cdbs/www-data/pdf/ATV0000/ATV0000CE5.pdf")
     (tags "SMD SMT SPST EVQPUM EVQPUD")
@@
   )
   (footprint "Connector_PinHeader_2.54mm:PinHeader_1x04_P2.54mm_Horizontal" (layer "F.Cu")
-    (at 14.3256 -3.8608)
+    (at 16.1544 -3.81)
     (descr "Through hole angled pin header, 1x04, 2.54mm pitch, 6mm pin length, single row")
     (tags "Through hole angled pin header THT 1x04 2.54mm single row")
@@
     )
   )
-  (gr_circle (center 0 0) (end 19 0)
+  (gr_circle (center 0 0) (end 21 0)
     (stroke (width 0.15) (type default)) (fill none) (layer "Edge.Cuts"))
 )
