File: HW/i2cExplorer/i2cExplorer.kicad_sch (KiCad schematic)
At the start: 19 parts, among them J1 GC9A01, J2 SWDIO, J3 I2CTest, J4 USB_C_Receptacle, Q1 S8050, SW1 SW_Push, SW2 SW_Push, SW3 SW_Push, U1 RP2040, U2 W5Q16JVSSIQ, Y1 Crystal

Commit message: update sch
Parts:
- added C1, C13, C14, C15, C16, C2, C6, C8, C9: 0.1uF, Capacitor_SMD:C_0603_1608Metric, symbol Device:C
- added C10, C12: 4.7uF, Capacitor_SMD:C_0603_1608Metric, symbol Device:C
- added C11: 120pF, Capacitor_SMD:C_0603_1608Metric, symbol Device:C
- added C3, C4: 10uF, Capacitor_SMD:C_0805_2012Metric, symbol Device:C
- added C5: 2.2uF, Capacitor_SMD:C_0603_1608Metric, symbol Device:C
- added C7: C, Capacitor_SMD:C_0603_1608Metric, symbol Device:C
- added R10: 0R2, Resistor_SMD:R_0603_1608Metric, symbol Device:R
- added R11, R12, R15: 1K, Resistor_SMD:R_0603_1608Metric, symbol Device:R
- added R13, R14, R18: 33K, Resistor_SMD:R_0603_1608Metric, symbol Device:R
- added R16, R22, R29, R30, R6: 100K, Resistor_SMD:R_0603_1608Metric, symbol Device:R
- added R17: 133K, Resistor_SMD:R_0603_1608Metric, symbol Device:R
- added R19: 102K, Resistor_SMD:R_0603_1608Metric, symbol Device:R
- added R20, R24, R25, R26, R33, R34, R4, R8: 330R, Resistor_SMD:R_0603_1608Metric, symbol Device:R
- added R21, R23, R27, R28, R31, R32, R5, R7: 1M, Resistor_SMD:R_0603_1608Metric, symbol Device:R
- added R9: 18KR, Capacitor_SMD:C_0603_1608Metric, symbol Device:R
- added U3, U7, U8, U9: SN74LVC1T45DBV, Package_TO_SOT_SMD:SOT-23-6, symbol Logic_LevelTranslator:SN74LVC1T45DBV
- added U4: MIC2025-1YM, Package_SO:SOIC-8_3.9x4.9mm_P1.27mm, symbol Power_Management:MIC2025-1YM
- added U5: GS6002, Package_SO:SOIC-8_3.9x4.9mm_P1.27mm, symbol Amplifier_Operational:AD8620
- added U6: AP2127K-ADJ, Package_TO_SOT_SMD:SOT-23-5, symbol Regulator_Linear:AP2127K-ADJ
- added U?: PW1502A, Package_TO_SOT_SMD:SOT-23-5, symbol Power_Protection:PW1502A
Connections:
- new net: C5.1, C6.1, U5.8 (V+)
- new net: R20.2, R21.2, U7.3 (A)
- new net: R29.2, U8.5 (DIR)
- new net: R11.1, R13.1, U5.3 (+)
- new net: C11.2, R17.2, R18.1, R19.1, U6.4 (ADJ)
- new net: C7.2, R15.1, U5.5 (+)
- new net: R9.1, U?.3 (IADJ)
- new net: R26.2, R28.2, U9.3 (A)
- new net: R32.2, R34.1, U9.4 (B)
- new net: R30.2, U9.5 (DIR)
- new net: R31.2, R33.1, U8.4 (B)
- new net: R23.2, R24.1, U7.4 (B)
- new net: R4.2, R5.2, U3.3 (A)
- new net: R7.2, R8.1, U3.4 (B)
- new net: R6.2, U3.5 (DIR)
- new net: R12.1, R14.2, U5.2 (-)
- new net: R22.2, U7.5 (DIR)
- new net: R25.2, R27.2, U8.3 (A)
- new net: U4.6 (OUT), U4.8 (OUT)
- new net +3V3: C1.1, C13.1, C14.1, C8.1, U3.1 (VCCA), U7.1 (VCCA), U8.1 (VCCA), U9.1 (VCCA)
- new net +VUSB: R10.2, R11.2
- new net 5V/2A: C3.1, U?.4 (EN), U?.5 (VIN)
- new net BUFIO_1: R20.1, R25.1, R26.1, R4.1
- new net BUF_OUT_1: R24.2, R33.2, R34.2, R8.2
- new net CURRENT_SENSE: R14.1, U5.1
- new net GND: C1.2, C10.2, C12.2, C13.2, C14.2, C15.2, C16.2, C2.2, C3.2, C5.2, C6.2, C7.1, C8.2, C9.2, R13.2, R16.2, R18.2, R21.1, R22.1, R23.1, R27.1, R28.1, R29.1, R30.1, R31.1, R32.1, R5.1, R6.1, R7.1, R9.2, U3.2 (GND), U5.4 (V-), U6.2 (GND), U7.2 (GND), U8.2 (GND), U9.2 (GND), U?.2 (GND)
- new net PWM_VREG_ADJ: R15.2
- new net USB2_5V/400mA: C4.1, U?.1 (VOUT)
- new net VREF_VOUT: C15.1, C16.1, C2.1, C9.1, U3.6 (VCCB), U7.6 (VCCB), U8.6 (VCCB), U9.6 (VCCB)
- new net VREG_ADJ: R19.2, U5.6 (-), U5.7
- new net VREG_EN: R16.1, U6.3 (EN)
- new net VREG_IN: C10.1, R10.1, R12.2, U6.1 (VIN)
- new net VREG_OUT: C11.1, C12.1, R17.1, U6.5 (VOUT)
Other:
- moved on the sheet: H1, H2, H3, H4, J1, J2, J3, J4, Q1, R2, R3, SW1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
